File: PSoCArtyShield.kicad_sch (KiCad schematic)
At the start: 15 parts, among them J1 Arty_Analog, J2 Arty_IOH, J3 Arty_I2C, J4 Arty_IOL, J5 Arty_XADC, J6 Arty_SPI, J7 Arty_Power

Commit message: wip
Parts:
- removed D?: 1N914WT, Diode_SMD:D_SOD-523, symbol Diode:1N914WT
- removed J?: DIN-5_180degree, symbol Connector:DIN-5_180degree
- removed R?: 1k, symbol Device:R
- removed R?: 220, symbol Device:R
- removed U?: LTV-357T, Package_SO:SO-4_4.4x3.6mm_P2.54mm, symbol Isolator:LTV-357T
- removed U?: S27KL0641DABHA020, BGA:BGA24_6x8x1.0mm_VAA024, symbol Memory:S27KL0641DABHA020
- added C1, C2, C3, C4, C5: 0.1uF, Capacitor_SMD:C_0402_1005Metric_Pad0.74x0.62mm_HandSolder, symbol Device:C
- added D0, D1, D2, D3, D4, D5, D6: LED, LED_SMD:LED_0603_1608Metric_Pad1.05x0.95mm_HandSolder, symbol Device:LED
- added J8, J9: Conn_01x03, Connector_PinHeader_2.54mm:PinHeader_1x03_P2.54mm_Vertical, symbol Connector_Generic:Conn_01x03
- added R0, R1, R2, R3, R4, R5, R6: R, Resistor_SMD:R_0603_1608Metric_Pad0.98x0.95mm_HandSolder, symbol Device:R
- added R10, R11, R7, R8, R9: 6.19k, Resistor_SMD:R_0603_1608Metric_Pad0.98x0.95mm_HandSolder, symbol Device:R
- added RV0, RV1, RV2, RV3: 10k, Potentiometer_THT:Potentiometer_Bourns_PTV09A-1_Single_Vertical, symbol Device:R_Potentiometer
- added SW0, SW1, SW2, SW3: SW_Push, Button_Switch_THT:SW_PUSH-12mm_Wuerth-430476085716, symbol Switch:SW_Push
- added SW4: RotaryEncoder, Rotary_Encoder:RotaryEncoder_Alps_EC11E_Vertical_H20mm, symbol Device:RotaryEncoder
- added TP0, TP1, TP10, TP2, TP3, TP4, TP5, TP6: ~, TestPoint:TestPoint_Keystone_5019_Minature, symbol Connector:TestPoint
- added TP7: Conn_01x08, Connector_PinHeader_2.54mm:PinHeader_1x08_P2.54mm_Vertical, symbol Connector_Generic:Conn_01x08
- added TP8: ~, Connector_PinHeader_2.54mm:PinHeader_1x01_P2.54mm_Vertical, symbol Connector_Generic:Conn_01x01
- added TP9: ~, Connector_PinHeader_2.54mm:PinHeader_1x08_P2.54mm_Vertical, symbol Connector_Generic:Conn_01x08
- J1: footprint (none) -> Connector_PinHeader_2.54mm:PinHeader_2x06_P2.54mm_Vertical
- J2, J4: footprint (none) -> Connector_PinHeader_2.54mm:PinHeader_2x08_P2.54mm_Vertical
- J3: footprint (none) -> Connector_PinHeader_2.54mm:PinHeader_1x02_P2.54mm_Vertical
- J5: footprint (none) -> Connector_PinHeader_2.54mm:PinHeader_2x02_P2.54mm_Vertical
- J6: footprint (none) -> Connector_PinHeader_2.54mm:PinHeader_2x03_P2.54mm_Vertical
- J7: footprint (none) -> Connector_PinHeader_2.54mm:PinHeader_1x08_P2.54mm_Vertical
- U1: renamed from U?; footprint (none) -> ProjectLibrary:CY8CKIT-059
- gave numbers to parts that had none: 1
Connections:
- net midi_rx is gone; now on net debug_rx: U1.1 (P2[0])
- net +3V3: now also X1.4 (VDD), C1.1, R10.1, R11.1, R7.1, R8.1, R9.1
- net GND: now also C1.2, C2.2, C3.2, C4.2, C5.2, D0.1 (K), D1.1 (K), D2.1 (K), D3.1 (K), J8.1 (Pin_1), J9.3 (Pin_3), R4.2, R5.2, R6.2, RV0.3, RV1.3, RV2.3, RV3.3, SW0.2, SW1.2, SW2.2, SW3.2, SW4.C, TP10.1, TP6.1, TP8.1 (Pin_1)
- net arty_cs: now also U1.16 (12[0]); no longer U1.24 (P1[7])
- net arty_miso: now also U1.13 (12[3]); no longer U1.21 (P1[4])
- net arty_mosi: now also U1.14 (12[2]); no longer U1.22 (P1[5])
- net arty_sck: now also U1.15 (12[1]); no longer U1.23 (P1[6])
- net arty_scl: no longer U1.20 (P1[3])
- net arty_sda: no longer U1.19 (P1[2])
- net debug_rx: now also J8.2 (Pin_2); no longer U1.4 (P2[3])
- net debug_tx: now also U1.4 (P2[3]), J8.3 (Pin_3); no longer U1.5 (P2[4])
- net i2s_sclk: now also U1.48 (P3[3]); no longer U1.49 (P3[2])
- net i2s_sdi: now also U1.46 (P3[5]); no longer U1.47 (P3[4])
- net i2s_sdo: now also U1.47 (P3[4]); no longer U1.48 (P3[3])
- net psoc_io7: now reaches J4.10 (Pin_10)
- net psoc_io7: now also U1.24 (P1[7]), TP9.8 (Pin_8)
- net fpga_led0: now reaches J4.12 (Pin_12)
- net fpga_led0: now also D4.2 (A)
- net fpga_led1: now reaches J4.14 (Pin_14)
- net fpga_led1: now also D5.2 (A)
- net fpga_led2: now reaches J4.16 (Pin_16)
- net fpga_led2: now also D6.2 (A)
- net psoc_io3: now reaches J4.2 (Pin_2)
- net psoc_io3: now also U1.20 (P1[3]), TP9.4 (Pin_4)
- net psoc_io4: now reaches J4.4 (Pin_4)
- net psoc_io4: now also U1.21 (P1[4]), TP9.5 (Pin_5)
- net psoc_io5: now reaches J4.6 (Pin_6)
- net psoc_io5: now also U1.22 (P1[5]), TP9.6 (Pin_6)
- net psoc_io6: now reaches J4.8 (Pin_8)
- net psoc_io6: now also U1.23 (P1[6]), TP9.7 (Pin_7)
- net psoc_led1: now reaches U1.10 (12[6])
- net psoc_led1: now also R1.2
- net psoc_led2: now reaches U1.11 (12[5])
- net psoc_led2: now also R2.2
- net psoc_led3: now reaches U1.12 (12[4])
- net psoc_led3: now also R3.2
- net psoc_io0: now reaches U1.17 (P1[0])
- net psoc_io0: now also J4.1 (Pin_1), TP9.1 (Pin_1)
- net psoc_io1: now reaches U1.18 (P1[1])
- net psoc_io1: now also J4.3 (Pin_3), TP9.2 (Pin_2)
- net ext_pot: now reaches U1.30 (P0[7])
- net ext_pot: now also J9.2 (Pin_2)
- net pot3: now reaches U1.31 (P0[6])
- net pot3: now also C5.1, RV3.2
- net pot2: now reaches U1.32 (P0[5])
- net pot2: now also C4.1, RV2.2
- net pot1: now reaches U1.36 (P0[1])
- net pot1: now also C3.1, RV1.2
- net pot0: now reaches U1.37 (P0[0])
- net pot0: now also C2.1, RV0.2
- net sw1: now reaches U1.6 (P2[5])
- net sw1: now also SW1.1
- net sw2: now reaches U1.7 (P2[6])
- net sw2: now also SW2.1
- net sw3: now reaches U1.8 (P2[7])
- net sw3: now also SW3.1
- net psoc_led0: now reaches U1.9 (12[7])
- net psoc_led0: now also R0.2
- net at J2.11 (Pin_11): now also TP5.1
- net gpio_0 renamed encb
- net encb: now also SW4.B; no longer J4.1 (Pin_1)
- net gpio_1 renamed enca
- net enca: now also SW4.A; no longer J4.3 (Pin_3)
- net gpio_2 renamed psoc_io2
- net psoc_io2: now also U1.19 (P1[2]), TP9.3 (Pin_3); no longer U1.46 (P3[5])
- net ram_ck: no longer names the net of J2.5 (Pin_5)
- net ram_ck: now also TP2.1
- net ram_dq0: no longer names the net of J2.2 (Pin_2)
- net ram_dq0: now also TP7.1 (Pin_1)
- net ram_dq1: no longer names the net of J2.4 (Pin_4)
- net ram_dq1: now also TP7.2 (Pin_2)
- net ram_dq2: no longer names the net of J2.6 (Pin_6)
- net ram_dq2: now also TP7.3 (Pin_3)
- net ram_dq3: no longer names the net of J2.8 (Pin_8)
- net ram_dq3: now also TP7.4 (Pin_4)
- net ram_dq4: no longer names the net of J2.10 (Pin_10)
- net ram_dq4: now also TP7.5 (Pin_5)
- net ram_dq5: no longer names the net of J2.12 (Pin_12)
- net ram_dq5: now also TP7.6 (Pin_6)
- net ram_dq6: no longer names the net of J2.14 (Pin_14)
- net ram_dq6: now also TP7.7 (Pin_7)
- net ram_dq7: no longer names the net of J2.16 (Pin_16)
- net ram_dq7: now also TP7.8 (Pin_8)
- net ram_rwds: no longer names the net of J2.9 (Pin_9)
- net ram_rwds: now also TP4.1
- net ~{ram_ck#}: no longer names the net of J2.7 (Pin_7)
- net ~{ram_ck#}: now also TP3.1
- net ~{ram_cs}: no longer names the net of J2.3 (Pin_3)
- net ~{ram_cs}: now also TP1.1
- net ~{ram_reset}: no longer names the net of J2.1 (Pin_1)
- net ~{ram_reset}: now also TP0.1
- new net: D4.1 (K), R4.1
- new net: D2.2 (A), R2.1
- new net: R10.2, RV3.1
- new net: R8.2, RV1.1
- new net: R7.2, RV0.1
- new net: D3.2 (A), R3.1
- new net: J9.1 (Pin_1), R11.2
- new net: D1.2 (A), R1.1
- new net: D0.2 (A), R0.1
- new net: D5.1 (K), R5.1
- new net: D6.1 (K), R6.1
- new net: R9.2, RV2.1
- new net sw0: SW0.1, U1.5 (P2[4])
- no-connect marks 9 -> 29
Other:
- note added: "External 10k pot"
- moved on the sheet: J1, J2
